Commit message: prepare robot pose ekf

File: chefbot_description/urdf/chefbot_rviz_base.urdf.xacro (robot description, xacro)
@@ -11,5 +11,5 @@
   <!-- Chefbot -->
   <xacro:macro name="kobuki">
-    <link name="base_footprint"/>
+    <!--link name="base_footprint"/-->
     <!--
        Base link is set at the bottom of the base mould.
@@ -21,9 +21,9 @@
        to 0.352.
       -->
-    <joint name="base_joint" type="fixed">
+    <!--joint name="base_joint" type="fixed">
       <origin xyz="0 0 0.0102" rpy="0 0 0" />
       <parent link="base_footprint"/>
       <child link="base_link" />
-    </joint>
+    </joint-->
     <link name="base_link">
       <visual>
